Commit message: Gazebo

File: description/robot.urdf.xacro (robot description, xacro)
@@ -2,3 +2,4 @@
 <robot xmlns:xacro="http://www.ros.org/wiki/xacro"  name="robot">
    <xacro:include filename="robot_core.xacro" />
+   <xacro:include filename="gazebo_control.xacro" />
 </robot>

File: description/robot_core.xacro (robot description, xacro)
@@ -39,4 +39,7 @@
         </xacro:inertial_box>
     </link>
+    <gazebo reference="chassis">
+    <material>Gazebo/White</material>
+    </gazebo>
         <!-- LEFT WHEEL LINK -->
     <joint name="left_wheel_joint" type="continuous">
@@ -62,4 +65,7 @@
         </xacro:inertial_cylinder>
     </link>
+    <gazebo reference="left_wheel">
+        <material>Gazebo/Blue</material>
+    </gazebo>
     <!-- RIGHT WHEEL LINK -->
     <joint name="right_wheel_joint" type="continuous">
@@ -85,4 +91,7 @@
         </xacro:inertial_cylinder>
     </link>
+     <gazebo reference="right_wheel">
+        <material>Gazebo/Blue</material>
+    </gazebo>
     <!-- CASTER WHEEL LINK -->
     <joint name="caster_wheel_joint" type="continuous">
@@ -107,3 +116,8 @@
         </xacro:inertial_sphere>
     </link>
+    <gazebo reference="caster_wheel">
+        <material>Gazebo/Black</material>
+        <mu1 value="0.001"/>
+        <mu2 value="0.001"/>
+    </gazebo>
 </robot>

Commit message: Lidar

File: description/robot.urdf.xacro (robot description, xacro)
@@ -3,3 +3,4 @@
    <xacro:include filename="robot_core.xacro" />
    <xacro:include filename="gazebo_control.xacro" />
+   <xacro:include filename="lidar.xacro" />
 </robot>

File: description/robot_core.xacro (robot description, xacro)
@@ -32,13 +32,13 @@
             <material name="white"/>
         </visual>
-         <!-- <collision>
-            <origin xyz="0.7305 0 0.31115"/>
+        <collision>
+            <origin xyz="1.0225 0 0.254" rpy="0 0 0"/>
             <geometry>
                 <box size="0.635 0.584 0.508"/>
             </geometry>
         </collision>
-        <xacro:inertial_box mass="0.5" x="0.3" y="0.5" z="0.15">
-                <origin xyz="0.15 0 0.075" rpy="0 0 0"/>
-        </xacro:inertial_box> -->
+        <xacro:inertial_box mass="0.5" x="0.635" y="0.584" z="0.508">
+            <origin xyz="1.0225 0 0.254" rpy="0 0 0"/>
+        </xacro:inertial_box>
     </link>
     <joint name="component_joint" type="fixed">
@@ -55,13 +55,13 @@
             <material name="blue"/>
         </visual>
-         <!-- <collision>
-            <origin xyz="0.7305 0 0.31115"/>
+         <collision>
+            <origin xyz="1.0225 0 0"/>
             <geometry>
                 <box size="0.635 0.584 0.1524"/>
             </geometry>
         </collision>
-        <xacro:inertial_box mass="0.5" x="0.635" y=".584" z=".1524">
+        <xacro:inertial_box mass="0.1" x="0.635" y=".584" z=".1524">
                 <origin xyz="1.0225 0 0" rpy="0 0 0"/>
-        </xacro:inertial_box> -->
+        </xacro:inertial_box>
     </link>
     <gazebo reference="chassis">
@@ -82,5 +82,6 @@
             <material name="red"/>
         </visual>
-         <!-- <collision>
+        <collision>
+            <origin xyz="0 0.3937 -1.2573"/>
             <geometry>
                  <cylinder radius="0.0889" length="2.27965" />
@@ -89,5 +90,5 @@
          <xacro:inertial_cylinder mass="0.1" radius="0.0889" length="2.27965" >
                 <origin xyz="0 0.3937 -1.2573" rpy="0 -${pi/2} 0"/>
-        </xacro:inertial_cylinder> -->
+        </xacro:inertial_cylinder>
     </link>
            <!-- RIGHT FLOAT LINK -->
@@ -105,5 +106,6 @@
             <material name="red"/>
         </visual>
-         <!-- <collision>
+         <collision>
+            <origin xyz="0 -0.3937 -1.2573"/>
             <geometry>
                  <cylinder radius="0.0889" length="2.27965" />
@@ -112,5 +114,76 @@
          <xacro:inertial_cylinder mass="0.1" radius="0.0889" length="2.27965" >
                 <origin xyz="0 -0.3937 -1.2573" rpy="0 -${pi/2} 0"/>
-        </xacro:inertial_cylinder> -->
+        </xacro:inertial_cylinder>
     </link>
+    <joint name="left_wheel_joint" type="continuous">
+        <parent link="chassis"/>
+        <child link="left_wheel"/>
+        <origin xyz="0.127 0.2411 0" rpy="-${pi/2} 0 0"/>
+        <axis xyz="0 0 1"/>
+    </joint>
+    <link name="left_wheel">
+    <visual>
+        <geometry>
+            <cylinder length="0.1" radius="0.127" />
+        </geometry>
+        <material name="blue"/>
+    </visual>
+    <collision>
+        <geometry>
+            <sphere  radius="0.127" />
+        </geometry>
+    </collision>
+    <xacro:inertial_sphere mass="0.1"  radius="0.127">
+       <origin xyz="0 0 0" rpy="0 0 0"/>
+    </xacro:inertial_sphere>
+    </link>
+    <joint name="right_wheel_joint" type="continuous">
+        <parent link="chassis"/>
+        <child link="right_wheel"/>
+        <origin xyz="0.127 -0.2411 0" rpy="${pi/2} 0 0"/>
+        <axis xyz="0 0 -1"/>
+    </joint>
+    <link name="right_wheel">
+    <visual>
+        <geometry>
+            <cylinder length="0.1" radius="0.127" />
+        </geometry>
+        <material name="blue"/>
+    </visual>
+    <collision>
+        <geometry>
+            <sphere  radius="0.127" />
+        </geometry>
+    </collision>
+    <xacro:inertial_sphere mass="0.1"  radius="0.127">
+       <origin xyz="0 0 0" rpy="0 0 0"/>
+    </xacro:inertial_sphere>
+    </link>
+<!-- CASTER WHEEL -->
+<joint name="caster_wheel_joint" type="continuous">
+    <parent link="chassis"/>
+    <child link="caster_wheel"/>
+    <origin xyz="1.0225 0 0" rpy="0 0 0"/>
+</joint>
+<link name="caster_wheel">
+    <visual>
+        <geometry>
+            <sphere radius="0.127" />
+        </geometry>
+        <material name="black"/>
+    </visual>
+    <collision>
+        <geometry>
+            <sphere  radius="0.127" />
+        </geometry>
+    </collision>
+    <xacro:inertial_sphere mass="0.05" radius="0.127">
+        <origin xyz="0 0 0" rpy="0 0 0"/>
+    </xacro:inertial_sphere>
+</link>
+<gazebo reference="caster_wheel">
+    <material>Gazebo/Black</material>
+    <mu1 value="0.001"/>
+    <mu2 value="0.001"/>
+</gazebo>
 </robot>

Commit message: controller-sim

File: description/robot.urdf.xacro (robot description, xacro)
@@ -3,4 +3,5 @@
    <xacro:include filename="robot_core.xacro" />
    <xacro:arg name="use_ros2_control" default="true"/>
+   <xacro:arg name="sim_mode" default="false"/>
    <xacro:if value="$(arg use_ros2_control)">
       <xacro:include filename="ros2_control.xacro" />

File: description/ros2_control.xacro (robot description, xacro)
@@ -1,58 +1,63 @@
 <?xml version="1.0"?>
 <robot xmlns:xacro="http://www.ros.org/wiki/xacro">
-<ros2_control name="RealRobot" type="system">
-    <hardware>
-        <plugin>diffdrive_arduino/DiffDriveArduino</plugin>
-        <param name="left_wheel_name">left_wheel_joint</param>
-        <param name="right_wheel_name">right_wheel_joint</param>
-        <param name="loop_rate">30</param>
-        <param name="device">/dev/ttyUSB0</param>
-        <param name="baud_rate">57600</param>
-        <param name="timeout">1000</param>
-        <param name="enc_counts_per_rev">1350</param>
-    </hardware>
-    <!-- Note everything below here is the same as the Gazebo one -->
-    <joint name="left_wheel_joint">
-        <command_interface name="velocity">
-            <param name="min">-10</param>
-            <param name="max">10</param>
-        </command_interface>
-        <state_interface name="velocity"/>
-        <state_interface name="position"/>
-    </joint>
-    <joint name="right_wheel_joint">
-        <command_interface name="velocity">
-            <param name="min">-10</param>
-            <param name="max">10</param>
-        </command_interface>
-        <state_interface name="velocity"/>
-        <state_interface name="position"/>
-    </joint>
-</ros2_control>
-    <!-- <ros2_control name="GazeboSystem" type="system">
-    <hardware>
-        <plugin>gazebo_ros2_control/GazeboSystem</plugin>
-    </hardware>
-    <joint name="left_wheel_joint">
-        <command_interface name="velocity">
-            <param name="min">-10</param>
-            <param name="max">10</param>
-        </command_interface>
-        <state_interface name="position" />
-        <state_interface name="velocity" />
-    </joint>
-    <joint name="right_wheel_joint">
-        <command_interface name="velocity">
-            <param name="min">-10</param>
-            <param name="max">10</param>
-        </command_interface>
-        <state_interface name="velocity" />
-        <state_interface name="position" />
-    </joint>
-    </ros2_control> -->
-<!-- <gazebo>
-    <plugin filename="libgazebo_ros2_control.so" name="gazebo_ros2_control">
-       <parameters>$(find my_bot)/config/my_controllers.yaml</parameters>
-    </plugin>
-</gazebo> -->
+<xacro:unless value="$(arg sim_mode)">
+            <ros2_control name="RealRobot" type="system">
+                <hardware>
+                    <plugin>diffdrive_arduino/DiffDriveArduino</plugin>
+                    <param name="left_wheel_name">left_wheel_joint</param>
+                    <param name="right_wheel_name">right_wheel_joint</param>
+                    <param name="loop_rate">30</param>
+                    <param name="device">/dev/ttyUSB0</param>
+                    <param name="baud_rate">57600</param>
+                    <param name="timeout">1000</param>
+                    <param name="enc_counts_per_rev">1350</param>
+                </hardware>
+                <!-- Note everything below here is the same as the Gazebo one -->
+                <joint name="left_wheel_joint">
+                    <command_interface name="velocity">
+                        <param name="min">-10</param>
+                        <param name="max">10</param>
+                    </command_interface>
+                    <state_interface name="velocity"/>
+                    <state_interface name="position"/>
+                </joint>
+                <joint name="right_wheel_joint">
+                    <command_interface name="velocity">
+                        <param name="min">-10</param>
+                        <param name="max">10</param>
+                    </command_interface>
+                    <state_interface name="velocity"/>
+                    <state_interface name="position"/>
+                </joint>
+            </ros2_control>
+ </xacro:unless>
+<xacro:if value="$(arg sim_mode)">
+            <ros2_control name="GazeboSystem" type="system">
+            <hardware>
+                <plugin>gazebo_ros2_control/GazeboSystem</plugin>
+            </hardware>
+            <joint name="left_wheel_joint">
+                <command_interface name="velocity">
+                    <param name="min">-10</param>
+                    <param name="max">10</param>
+                </command_interface>
+                <state_interface name="position" />
+                <state_interface name="velocity" />
+            </joint>
+            <joint name="right_wheel_joint">
+                <command_interface name="velocity">
+                    <param name="min">-10</param>
+                    <param name="max">10</param>
+                </command_interface>
+                <state_interface name="velocity" />
+                <state_interface name="position" />
+            </joint>
+            </ros2_control>
+</xacro:if>
+            <gazebo>
+                <plugin filename="libgazebo_ros2_control.so" name="gazebo_ros2_control">
+                <parameters>$(find my_bot)/config/my_controllers.yaml</parameters>
+                 <parameters>$(find my_bot)/config/gaz_ros2_ctl_use_sim.yaml</parameters>
+                </plugin>
+            </gazebo>
 </robot>
